Commit message: Loaded real environment

File: src/smr1_moveit_config/urdf/workcell.xacro (robot description, xacro)
@@ -3,27 +3,23 @@
     <xacro:include filename="$(find ur_description)/urdf/ur5.urdf.xacro" />
     <xacro:ur5_robot prefix="" joint_limited="true"/>
-    <joint name="table_to_robot" type="fixed">
-        <parent link="table"/>
+    <joint name="env_to_robot" type="fixed">
+        <parent link="env"/>
         <child link="base_link"/>
-        <origin xyz="0 0 0" rpy="0 0 0"/>
+        <origin xyz="-0.85 -0.42 1.55" rpy="0 0 0"/>
     </joint>
     <link name="world"/>
-    <link name="table">
+    <link name="env" >
         <visual>
             <geometry>
-                <box size="1.0 1.0 0.05"/>
+                <mesh filename="package://smr1_moveit_config/urdf/smrsetup.stl"/>
             </geometry>
+            <origin xyz="0 0 0" rpy="3.14 0 3.14" />
         </visual>
-        <collision>
-            <geometry>
-                <box size="1.0 1.0 0.05"/>
-            </geometry>
-        </collision>
     </link>
     <link name="camera_frame"/>
-    <joint name="world_to_table" type="fixed">
-        <parent link="world"/>
-        <child link="table"/>
-        <origin xyz="0 0 0.5" rpy="0 0 0"/>
+    <joint name="world_to_env" type="fixed">
+        <parent link="world" />
+        <child link ="env" />
+        <origin xyz="0 0 0" rpy="0 0 0" />
     </joint>
     <joint name="world_to_camera" type="fixed">

Commit message: Added EOAT in moveit

File: src/smr1_moveit_config/urdf/workcell.xacro (robot description, xacro)
@@ -8,4 +8,9 @@
         <origin xyz="-0.85 -0.42 1.55" rpy="0 0 0"/>
     </joint>
+    <joint name="eoat_to_tool0" type="fixed">
+        <parent link="tool0" />
+        <child link="eoat" />
+        <origin xyz="0 0 0" rpy="0 0 -2.36"/>
+    </joint>
     <link name="world"/>
     <link name="env" >
@@ -15,4 +20,11 @@
             </geometry>
             <origin xyz="0 0 0" rpy="3.14 0 3.14" />
+        </visual>
+    </link>
+    <link name="eoat">
+        <visual>
+            <geometry>
+                <mesh filename="package://smr1_moveit_config/urdf/eoat.stl" />
+            </geometry>
         </visual>
     </link>

Commit message: Updated moveit config

File: src/smr1_moveit_config/urdf/workcell.xacro (robot description, xacro)
@@ -1,4 +1,10 @@
 <?xml version="1.0" ?>
 <robot name="myworkcell" xmlns:xacro="http://ros.org/wiki/xacro">
+    <material name="blue">
+        <color rgba="0 0 0.8 1" />
+    </material>
+    <material name="white">
+        <color rgba="1 1 1 1" />
+    </material>
     <xacro:include filename="$(find ur_description)/urdf/ur5.urdf.xacro" />
     <xacro:ur5_robot prefix="" joint_limited="true"/>
@@ -20,4 +26,5 @@
             </geometry>
             <origin xyz="0 0 0" rpy="3.14 0 3.14" />
+            <material name="blue" />
         </visual>
     </link>
@@ -27,4 +34,5 @@
                 <mesh filename="package://smr1_moveit_config/urdf/eoat.stl" />
             </geometry>
+            <material name="white" />
         </visual>
     </link>

Commit message: Added ur_modern_driver, moved ur5 to actual position

File: src/smr1_moveit_config/urdf/workcell.xacro (robot description, xacro)
@@ -12,5 +12,5 @@
         <parent link="env"/>
         <child link="base_link"/>
-        <origin xyz="-0.85 -0.42 1.55" rpy="0 0 0"/>
+        <origin xyz="-0.75 -0.52 1.57" rpy="0 0 0"/>
     </joint>
     <joint name="eoat_to_tool0" type="fixed">

Commit message: Edited pickup movement

File: src/smr1_moveit_config/urdf/workcell.xacro (robot description, xacro)
@@ -17,5 +17,5 @@
         <parent link="tool0" />
         <child link="eoat" />
-        <origin xyz="0 0 0" rpy="0 0 -2.36"/>
+        <origin xyz="0 0 0" rpy="0 0 0.84"/>
     </joint>
     <link name="world"/>
@@ -34,4 +34,5 @@
                 <mesh filename="package://smr1_moveit_config/urdf/eoat.stl" />
             </geometry>
+             <origin xyz="0 0 0" rpy="0 0 0" />
             <material name="white" />
         </visual>

Commit message: Added Collision Mashes to the enviroment

File: src/smr1_moveit_config/urdf/workcell.xacro (robot description, xacro)
@@ -12,5 +12,5 @@
         <parent link="env"/>
         <child link="base_link"/>
-        <origin xyz="-0.75 -0.52 1.57" rpy="0 0 0"/>
+        <origin xyz="0.085 0.355 0.880" rpy="0 0 3.14"/>
     </joint>
     <joint name="eoat_to_tool0" type="fixed">
@@ -19,13 +19,45 @@
         <origin xyz="0 0 0" rpy="0 0 0.84"/>
     </joint>
-    <link name="world"/>
+    <link name="world" />
     <link name="env" >
         <visual>
             <geometry>
-                <mesh filename="package://smr1_moveit_config/urdf/smrsetup.stl"/>
+                <mesh filename="package://smr1_moveit_config/urdf/Conveyor_belt.stl"/>
             </geometry>
-            <origin xyz="0 0 0" rpy="3.14 0 3.14" />
+            <origin xyz="-0.73 -0.02 0.666" rpy="1.57 0 0.0" />
             <material name="blue" />
         </visual>
+        <collision>
+            <geometry>
+                <box size="3.01 0.44 0.845"/>
+            </geometry>
+            <origin xyz="-0.73 -0.22 0.3225" rpy="0 0 0.0" />
+        </collision>
+        <visual>
+            <geometry>
+                <mesh filename="package://smr1_moveit_config/urdf/Tafel.stl"/>
+            </geometry>
+            <origin xyz="1.0 0.35 0" rpy="0 0 3.14" />
+            <material name="blue" />
+        </visual>
+        <collision>
+            <geometry>
+                <box size="2.0 0.70 0.860"/>
+            </geometry>
+            <origin xyz="1.0 0.35 0.43" rpy="0 0 0.0" />
+        </collision>
+        <visual>
+            <geometry>
+                <box size="4.0 0.10 3.0"/>
+            </geometry>
+            <origin xyz="0.0 0.76 1.5" rpy="0 0 0" />
+            <material name="blue" />
+        </visual>
+        <collision>
+            <geometry>
+                <box size="4.0 0.10 3.0"/>
+            </geometry>
+            <origin xyz="0.0 0.76 1.5" rpy="0 0 0" />
+        </collision>
     </link>
     <link name="eoat">

Commit message: Working orientation constraints

File: src/smr1_moveit_config/urdf/workcell.xacro (robot description, xacro)
@@ -10,5 +10,5 @@
     <xacro:ur5_robot prefix="" joint_limited="true"/>
     <joint name="env_to_robot" type="fixed">
-        <parent link="env"/>
+        <parent link="world"/>
         <child link="base_link"/>
         <origin xyz="0.085 0.355 0.880" rpy="0 0 3.14"/>
@@ -17,5 +17,5 @@
         <parent link="tool0" />
         <child link="eoat" />
-        <origin xyz="0 0 0" rpy="0 0 0.84"/>
+        <origin xyz="0 0 0" rpy="0 0 0"/>
     </joint>
     <link name="world" />
@@ -30,5 +30,5 @@
         <collision>
             <geometry>
-                <box size="3.01 0.44 0.845"/>
+                <box size="3.01 0.44 0.846"/>
             </geometry>
             <origin xyz="-0.73 -0.22 0.3225" rpy="0 0 0.0" />
@@ -66,5 +66,5 @@
                 <mesh filename="package://smr1_moveit_config/urdf/eoat.stl" />
             </geometry>
-             <origin xyz="0 0 0" rpy="0 0 0" />
+             <origin xyz="0 0 0" rpy="0 0 0.78" />
             <material name="white" />
         </visual>

Commit message: Collision constrains working better Added plant collision object after picking up plant

File: src/smr1_moveit_config/urdf/workcell.xacro (robot description, xacro)
@@ -30,7 +30,7 @@
         <collision>
             <geometry>
-                <box size="3.01 0.44 0.846"/>
+                <box size="3.01 0.44 0.860"/>
             </geometry>
-            <origin xyz="-0.73 -0.22 0.3225" rpy="0 0 0.0" />
+                <origin xyz="-0.73 -0.22 0.3225" rpy="0 0 0.0" />
         </collision>
         <visual>
@@ -58,6 +58,12 @@
                 <box size="4.0 0.10 3.0"/>
             </geometry>
-            <origin xyz="0.0 0.76 1.5" rpy="0 0 0" />
+            <origin xyz="0.0 -0.55 1.5" rpy="0 0 0" />
         </collision>
+        <collision>
+                    <geometry>
+                        <box size="4.0 0.10 3.0"/>
+                    </geometry>
+                    <origin xyz="0.0 0.76 1.5" rpy="0 0 0" />
+                </collision>
     </link>
     <link name="eoat">

Commit message: Update

File: src/smr1_moveit_config/urdf/workcell.xacro (robot description, xacro)
@@ -12,5 +12,5 @@
         <parent link="world"/>
         <child link="base_link"/>
-        <origin xyz="0.085 0.355 0.880" rpy="0 0 3.14"/>
+        <origin xyz="0.0 0.0 0.880" rpy="0 0 3.14"/>
     </joint>
     <joint name="eoat_to_tool0" type="fixed">
@@ -25,5 +25,5 @@
                 <mesh filename="package://smr1_moveit_config/urdf/Conveyor_belt.stl"/>
             </geometry>
-            <origin xyz="-0.73 -0.02 0.666" rpy="1.57 0 0.0" />
+            <origin xyz="-1.265 0.61 0.666" rpy="1.57 0 0.0" />
             <material name="blue" />
         </visual>
@@ -32,11 +32,11 @@
                 <box size="3.01 0.44 0.860"/>
             </geometry>
-                <origin xyz="-0.73 -0.22 0.3225" rpy="0 0 0.0" />
+                <origin xyz="-1.265 0.41 0.3225" rpy="0 0 0.0" />
         </collision>
         <visual>
             <geometry>
-                <mesh filename="package://smr1_moveit_config/urdf/Tafel.stl"/>
+                <box size="2.0 0.70 0.860"/>
             </geometry>
-            <origin xyz="1.0 0.35 0" rpy="0 0 3.14" />
+            <origin xyz="0.0 -0.225 0.43" rpy="0 0 0" />
             <material name="blue" />
         </visual>
@@ -45,5 +45,5 @@
                 <box size="2.0 0.70 0.860"/>
             </geometry>
-            <origin xyz="1.0 0.35 0.43" rpy="0 0 0.0" />
+            <origin xyz="0.0 -0.225 0.44" rpy="0 0 0.0" />
         </collision>
         <visual>
@@ -51,5 +51,5 @@
                 <box size="4.0 0.10 3.0"/>
             </geometry>
-            <origin xyz="0.0 0.76 1.5" rpy="0 0 0" />
+            <origin xyz="0.0 0.73 1.5" rpy="0 0 0" />
             <material name="blue" />
         </visual>
@@ -58,23 +58,55 @@
                 <box size="4.0 0.10 3.0"/>
             </geometry>
-            <origin xyz="0.0 -0.55 1.5" rpy="0 0 0" />
+            <origin xyz="0.0 0.73 1.5" rpy="0 0 0" />
         </collision>
+        <visual>
+            <geometry>
+                <mesh filename="package://smr1_moveit_config/urdf/tray.stl"/>
+            </geometry>
+            <origin xyz="-0.75 0.09 0.86" rpy="1.57 0.0 0.0" />
+            <material name="blue" />
+        </visual>
         <collision>
-                    <geometry>
-                        <box size="4.0 0.10 3.0"/>
-                    </geometry>
-                    <origin xyz="0.0 0.76 1.5" rpy="0 0 0" />
-                </collision>
+            <geometry>
+                <mesh filename="package://smr1_moveit_config/urdf/tray.stl"/>
+            </geometry>
+            <origin xyz="-0.75 0.09 0.86" rpy="1.57 0.0 0.0" />
+        </collision>
+        <visual>
+            <geometry>
+                <mesh filename="package://smr1_moveit_config/urdf/tray.stl"/>
+            </geometry>
+            <origin xyz="0.50 0.09 0.86" rpy="1.57 0.0 0.0" />
+            <material name="blue" />
+        </visual>
+        <collision>
+            <geometry>
+                <mesh filename="package://smr1_moveit_config/urdf/tray.stl"/>
+            </geometry>
+            <origin xyz="0.50 0.09 0.86" rpy="1.57 0.0 0.0" />
+        </collision>
+        <visual>
+            <geometry>
+                <mesh filename="package://smr1_moveit_config/urdf/tray.stl"/>
+            </geometry>
+            <origin xyz="-0.285 -0.545 0.86" rpy="1.57 0.0 1.57" />
+            <material name="blue" />
+        </visual>
+        <collision>
+            <geometry>
+                <mesh filename="package://smr1_moveit_config/urdf/tray.stl"/>
+            </geometry>
+            <origin xyz="-0.285 -0.545 0.86" rpy="1.57 0.0 1.57" />
+        </collision>
     </link>
     <link name="eoat">
         <visual>
             <geometry>
-                <mesh filename="package://smr1_moveit_config/urdf/eoat.stl" />
+                <mesh filename="package://smr1_moveit_config/urdf/eoat_v2.stl" />
             </geometry>
-             <origin xyz="0 0 0" rpy="0 0 0.78" />
+             <origin xyz="0 0 0.17" rpy="-1.57 0 -2.35" />
             <material name="white" />
         </visual>
     </link>
-    <link name="camera_frame"/>
     <joint name="world_to_env" type="fixed">
         <parent link="world" />
@@ -82,8 +114,3 @@
         <origin xyz="0 0 0" rpy="0 0 0" />
     </joint>
-    <joint name="world_to_camera" type="fixed">
-        <parent link="world"/>
-        <child link="camera_frame"/>
-        <origin xyz="-0.25 -0.5 1.25" rpy="0 3.14159 0"/>
-    </joint>
 </robot>

Commit message: Update, Improved enviroment looks

File: src/smr1_moveit_config/urdf/workcell.xacro (robot description, xacro)
@@ -6,4 +6,16 @@
     <material name="white">
         <color rgba="1 1 1 1" />
+    </material>
+    <material name="black">
+            <color rgba="0.1 0.1 0.1 1" />
+    </material>
+    <material name="gray">
+            <color rgba="0.7 0.7 0.7 1" />
+    </material>
+    <material name="yellow">
+            <color rgba="0.9 0.8 0.3 1" />
+    </material>
+    <material name="poster">
+            <texture filename="package://smr1_moveit_config/poster.png"/>
     </material>
     <xacro:include filename="$(find ur_description)/urdf/ur5.urdf.xacro" />
@@ -34,4 +46,15 @@
                 <origin xyz="-1.265 0.41 0.3225" rpy="0 0 0.0" />
         </collision>
+    </link>
+    <link name="poster">
+        <visual>
+            <geometry>
+                <box size="1.5 1.059 0.0"/>
+            </geometry>
+             <origin xyz="2.0 0.0 -0.675" rpy="0 0 0" />
+            <material name="poster" />
+        </visual>
+    </link>
+    <link name="table">
         <visual>
             <geometry>
@@ -39,5 +62,5 @@
             </geometry>
             <origin xyz="0.0 -0.225 0.43" rpy="0 0 0" />
-            <material name="blue" />
+            <material name="yellow" />
         </visual>
         <collision>
@@ -47,4 +70,6 @@
             <origin xyz="0.0 -0.225 0.44" rpy="0 0 0.0" />
         </collision>
+    </link>
+    <link name="back_wall">
         <visual>
             <geometry>
@@ -52,5 +77,5 @@
             </geometry>
             <origin xyz="0.0 0.73 1.5" rpy="0 0 0" />
-            <material name="blue" />
+            <material name="gray" />
         </visual>
         <collision>
@@ -60,4 +85,6 @@
             <origin xyz="0.0 0.73 1.5" rpy="0 0 0" />
         </collision>
+    </link>
+    <link name="trays">
         <visual>
             <geometry>
@@ -65,5 +92,5 @@
             </geometry>
             <origin xyz="-0.75 0.09 0.86" rpy="1.57 0.0 0.0" />
-            <material name="blue" />
+            <material name="black" />
         </visual>
         <collision>
@@ -78,5 +105,5 @@
             </geometry>
             <origin xyz="0.50 0.09 0.86" rpy="1.57 0.0 0.0" />
-            <material name="blue" />
+            <material name="black" />
         </visual>
         <collision>
@@ -91,5 +118,5 @@
             </geometry>
             <origin xyz="-0.285 -0.545 0.86" rpy="1.57 0.0 1.57" />
-            <material name="blue" />
+            <material name="black" />
         </visual>
         <collision>
@@ -114,3 +141,23 @@
         <origin xyz="0 0 0" rpy="0 0 0" />
     </joint>
+    <joint name="world_to_table" type="fixed">
+        <parent link="world" />
+        <child link ="table" />
+        <origin xyz="0 0 0" rpy="0 0 0" />
+    </joint>
+    <joint name="world_to_back_wall" type="fixed">
+        <parent link="world" />
+        <child link ="back_wall" />
+        <origin xyz="0 0 0" rpy="0 0 0" />
+    </joint>
+    <joint name="world_to_trays" type="fixed">
+        <parent link="world" />
+        <child link ="trays" />
+        <origin xyz="0 0 0" rpy="0 0 0" />
+    </joint>
+    <joint name="world_to_poster" type="fixed">
+        <parent link="world" />
+        <child link ="poster" />
+        <origin xyz="0 0 0" rpy="0 -1.57 1.57" />
+    </joint>
 </robot>
